File: pcb/jamboard-R.kicad_pcb (KiCad board)
At the start: 2 copper layers, 141.5 x 117.8 mm, 117 parts, among them J3 RJ45, U2 Pico

Commit message: worked on readme
Parts:
- moved D34 2.24 mm to (203.5, 95.0)
- moved D17 1.14 mm to (165.6, 62.4)
- moved D1 0.86 mm to (127.8, 65.1)
- moved D33 0.73 mm to (204.1, 72.0)
- moved D2 0.63 mm to (128.0, 83.9)
- moved D28 0.39 mm to (185.4, 129.1)
- moved D50 0.37 mm to (128.5, 135.2)
- moved D36 0.33 mm to (204.5, 129.2)
- moved D4 0.20 mm to (128.1, 122.2)
- moved D3 0.10 mm to (128.1, 102.8)
Routing:
- net Net-(D59-DIN): track 0.00 -> 28.4 mm, vias 0 -> 2
- net R_MATRIX ROW 3: track 180.8 -> 183.7 mm
- net Net-(D34-A): track 7.90 -> 6.16 mm
- net R_MATRIX ROW 1: track 176.8 -> 178.3 mm
- net +5V: track 882.9 -> 884.4 mm
- net R_MATRIX ROW 0: track 224.5 -> 225.1 mm
- net Net-(D33-A): track 3.90 -> 3.46 mm, vias 0 -> 1
- net GND: vias 10 -> 21
